Commit message: untracked nav files

File: ros_ws/src/dexmate_vega_description/robots/humanoid/vega_1p/vega_1p_f5d6.urdf (robot description, URDF)
Before this commit: robot vega_1p_f5d6, 75 links, 74 joints
Joints:
- joint L_arm_j4: limit lower=-3.071 upper=0.244 effort=80 velocity=2.7 -> lower=-3.071 upper=0.0 effort=80 velocity=2.7
- joint R_arm_j4: limit lower=-3.071 upper=0.244 effort=80 velocity=2.7 -> lower=-3.071 upper=0.0 effort=80 velocity=2.7

File: ros_ws/src/dexmate_vega_description/robots/humanoid/vega_1p/vega_1p_f5d6_collision_spheres.collision.urdf (robot description, URDF)
Before this commit: robot vega_1p_f5d6, 75 links, 74 joints
Joints:
- joint L_arm_j4: limit lower=-3.071 upper=0.244 effort=80 velocity=2.7 -> lower=-3.071 upper=0.0 effort=80 velocity=2.7
- joint R_arm_j4: limit lower=-3.071 upper=0.244 effort=80 velocity=2.7 -> lower=-3.071 upper=0.0 effort=80 velocity=2.7
